Commit message: aubo_i7.urdf: joint 3 (foreArm) axis +z like i5
foreArm_Joint had axis 0 0 -1, so the i7 model bent joint 3 the opposite
way from the real arm. With +z the i7 FK matches the i5's at the same
joints (EE pointing down at home), scaled to i7 link lengths.

Co-Authored-By: Claude Opus 5.5 <noreply@anthropic.com>
Claude-Session: https://claude.ai/code/session_01KDq8D3ggCuTYw9KV7FHrTk

File: backend/robot_sim/aubo-i5-full-master/aubo_description/urdf/aubo_i7.urdf (robot description, URDF)
Before this commit: robot aubo_i7, 8 links, 7 joints
Joints:
- joint foreArm_Joint: axis 0 0 -1 -> 0 0 1
